File: charliepad.sch (KiCad schematic (older format))
At the start: 28 parts, among them J1 USB4105-GF-A, SW1 SW_PUSH, SW10 SW_PUSH, SW11 SW_PUSH, SW12 SW_PUSH, SW2 SW_PUSH, SW3 SW_PUSH, SW4 SW_PUSH, SW5 SW_PUSH, SW6 SW_PUSH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

Commit message: Regularize track width Re-layout all the things, add logos, simple fw
Parts:
- removed F1: 1206L050YR, footprints:PTC_1206, symbol 1206L050_15:1206L050_15
- added F1: Polyfuse 1206L050YR, footprints:PTC_1206, symbol Device:Polyfuse
Other:
- moved on the sheet: C1, C2, D1, D2, D3, D4, D5, D6, J1, R1, R2, R3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
